File: _autosave-e-key-slot.kicad_pcb (KiCad board)
At the start: 2 copper layers, 28 x 37.6 mm, 46 parts, among them J1 PJ-018, J2 MDT420E03002, Q1 TSM9409CS, Q2 TSM9409CS, Q3 TSM9409CS, Q4 SSM3J328R_LF, U1 TPS54331DRG4, U2 MCP73831T-5ACI_OT, U4 MT3608

Commit message: Add .gitignore
Signed-off-by: JeffMboya <jangina.mboya@gmail.com>
Routing:
- net VSENCE: vias 1 -> 0
- net Net-(J1-Pad1): vias 1 -> 0
- net Net-(D6-K): vias 1 -> 0
- net Net-(D1-PadC): vias 1 -> 0
- net Net-(D1-PadA): vias 1 -> 0
- net COMP: vias 1 -> 0
- net BOOT: vias 1 -> 0
- net (no net): vias 3 -> 0
Changed lines of the file:
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@@
 		(layer "Edge.Cuts")
-	)
-	(via
-		(at 99.7 82.1)
-		(size 0.6)
-		(drill 0.3)
-		(layers "F.Cu" "B.Cu")
-		(net 0)
-	)
-	(via
-		(at 99.4 83.6)
-		(size 0.6)
-		(drill 0.3)
-		(layers "F.Cu" "B.Cu")
-		(net 0)
-	)
-	(via
-		(at 102.5 82)
-		(size 0.6)
-		(drill 0.3)
-		(layers "F.Cu" "B.Cu")
-		(net 0)
 	)
 	(segment
@@
 		(net 2)
 	)
-	(via
-		(at 91 89.3)
-		(size 0.6)
-		(drill 0.3)
-		(layers "F.Cu" "B.Cu")
-		(free yes)
-		(net 2)
-	)
 	(segment
 		(start 92.5 55.725)
@@
 		(net 6)
 	)
-	(via
-		(at 106.4 82.1)
-		(size 0.6)
-		(drill 0.3)
-		(layers "F.Cu" "B.Cu")
-		(free yes)
-		(net 6)
-	)
 	(segment
 		(start 81.8 73.5)
@@
 		(net 14)
 	)
-	(via
-		(at 91 90.2)
-		(size 0.6)
-		(drill 0.3)
-		(layers "F.Cu" "B.Cu")
-		(free yes)
-		(net 14)
-	)
 	(segment
 		(start 88.025 65.955)
@@
 		(net 15)
 	)
-	(via
-		(at 83 84.4)
-		(size 0.6)
-		(drill 0.3)
-		(layers "F.Cu" "B.Cu")
-		(free yes)
-		(net 15)
-	)
 	(segment
 		(start 85.17 85.6)
@@
 		(net 16)
 	)
-	(via
-		(at 85.7 83.2)
-		(size 0.6)
-		(drill 0.3)
-		(layers "F.Cu" "B.Cu")
-		(free yes)
-		(net 16)
-	)
 	(segment
 		(start 104.7 83.2)
@@
 		(net 18)
 	)
-	(via
-		(at 103.6 82.1)
-		(size 0.6)
-		(drill 0.3)
-		(layers "F.Cu" "B.Cu")
-		(free yes)
-		(net 18)
-	)
 	(segment
 		(start 95.6 88.2)
@@
 		(net 19)
 	)
-	(via
-		(at 97.6 88.2)
-		(size 0.6)
-		(drill 0.3)
-		(layers "F.Cu" "B.Cu")
-		(free yes)
-		(net 19)
-	)
