File: kicad/e-key-socket.kicad_sch (KiCad schematic)
At the start: 9 parts, among them J1 BM02B-SRSS-TB_LF__SN_, J2 MDT420E03002, U2 AZ1117IH-3.3TRG1

Commit message: Update tite block
Signed-off-by: JeffMboya <jangina.mboya@gmail.com>
Other:
- company: (none) -> Abstract Machines
- title: (none) -> M.2 E-Key Socket
Changed lines of the file:
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@@
 	(generator_version "8.0")
 	(paper "A4")
+	(title_block
+		(title "M.2 E-Key Socket")
+		(date "22 NOV 2024")
+		(rev "4")
+		(company "Abstract Machines")
+		(comment 1 "Drawn by: Jeff Mboya")
+		(comment 2 "Approved by:")
+	)
 	(junction
 		(at 59.69 83.82)
