File: kicad/am-iot-gateway.kicad_pcb (KiCad board)
At the start: 4 copper layers, 22 x 42 mm, 58 parts, among them J1 Bus_M.2_Socket_E, J3 GNSS Antenna, J4 RF Antenna, J5 NSIM-5-B, Q1 SS8050, Q2 SS8050, Q3 SS8050, SW1 SW_Push, U1 ESP32-C6-MINI-1/U, U2 SIM7080G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

Commit message: Place components on PCB
Signed-off-by: JeffMboya <jangina.mboya@gmail.com>
Parts:
- removed C3, C6: 1uF, Capacitor_SMD:C_0603_1608Metric
- removed C4, C5: 0.1uF, Capacitor_SMD:C_0603_1608Metric
- removed FID1, FID2, FID3, FID4, FID5, FID6: Fiducial, Fiducial:Fiducial_0.5mm_Mask1mm
- removed R2: 10K, Resistor_SMD:R_0603_1608Metric
- removed SW1: SW_Push, tactile-switch:SW4_PTS815 SJM 250 SMTR LFS_CNK
- removed TP1, TP2, TP3: TestPoint, TestPoint:TestPoint_Pad_D1.0mm
- removed U1: ESP32-C6-MINI-1/U, PCM_Espressif:ESP32-C6-MINI-1U
- C10, C11, C13, C14, C15, C16, D2, D4, Q1, Q2, Q3, R11, R12, R13, R14, R15, R16, R3, R4, R6, R9, U2, U3: moved to F.Cu
- J5: moved to B.Cu
- moved J4 32.5 mm to (85.8, 85.3)
- moved J3 31.5 mm to (99.5, 87.2), turned to 180 degrees
- moved D1 29.7 mm to (94.0, 56.5)
- moved R1 21.1 mm to (83.3, 85.6), turned to 90 degrees
- moved D2 19.7 mm to (84.9, 51.0), turned to 0 degrees
- moved R5 19.7 mm to (103.0, 85.8), turned to -90 degrees
- moved C13 17.3 mm to (85.5, 80.4)
- moved D3 17.2 mm to (99.5, 83.0)
- moved R15 17.1 mm to (87.4, 54.8), turned to 0 degrees
- moved R11 16.3 mm to (102.3, 53.1), turned to 180 degrees
- moved C10 15.9 mm to (103.0, 82.2)
- moved R8 14.0 mm to (83.3, 79.5)
- moved JP1 12.8 mm to (100.1, 79.0), turned to -90 degrees
- moved C14 12.3 mm to (87.9, 80.4)
- moved D4 12.1 mm to (101.5, 50.9), turned to 0 degrees
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Connections:
- J1 pad 20: M2_RXD(3v3) -> unconnected-(J1-~{UART_WAKE}-Pad20)
- J1 pad 22: M2_TXD(3v3) -> unconnected-(J1-UART_RXD-Pad22)
- J1 pad 3: USB_D+ -> unconnected-(J1-USB_D+-Pad3)
- J1 pad 5: USB_D- -> unconnected-(J1-USB_D--Pad5)
- J1 pad 59: MTMS -> unconnected-(J1-RESERVED/PETp1-Pad59)
- J1 pad 61: MTDI -> unconnected-(J1-RESERVED/PETn1-Pad61)
- J1 pad 65: MTCK -> unconnected-(J1-RESERVED/PERp1-Pad65)
- J1 pad 67: MTDO -> unconnected-(J1-RESERVED/PERn1-Pad67)
- U3 pad 15: M2_TXD(3v3) -> unconnected-(U3-B5-Pad15)
- U3 pad 16: M2_RXD(3v3) -> unconnected-(U3-B4-Pad16)
- U3 pad 5: M2_TXD -> unconnected-(U3-A4-Pad5)
- U3 pad 6: M2_RXD -> unconnected-(U3-A5-Pad6)
Routing:
- net GND: track 350.3 -> 0.00 mm, vias 4 -> 0
- net +1V8: track 93.1 -> 0.00 mm, vias 5 -> 0
- net +3V3: track 82.1 -> 0.00 mm, vias 3 -> 0
- net Net-(D2-K): track 41.3 -> 0.00 mm, vias 2 -> 0
- net SIM7080G_SDA: track 41.0 -> 0.00 mm, vias 2 -> 0
- net SIM_DATA: track 39.9 -> 0.00 mm, vias 3 -> 0
- net RF_ANT: track 39.8 -> 0.00 mm, vias 2 -> 0
- net SIM7080G_PWR: track 36.7 -> 0.00 mm, vias 2 -> 0
- net M2_TXD(3v3): track 35.3 -> 0.00 mm, vias 3 -> 0
- net M2_RXD(3v3): track 34.4 -> 0.00 mm, vias 4 -> 0
- net SIM7080G_TXD: track 33.6 -> 0.00 mm, vias 4 -> 0
- net SIM7080G_RXD: track 33.4 -> 0.00 mm, vias 3 -> 0
- net PWR_KEY: track 27.4 -> 0.00 mm, vias 2 -> 0
- net STATUS: track 23.6 -> 0.00 mm, vias 2 -> 0
- net SIM_CLK: track 22.4 -> 0.00 mm, vias 1 -> 0
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
Commit message: Route PCB
Signed-off-by: JeffMboya <jangina.mboya@gmail.com>
Routing:
- net GND: track 0.00 -> 185.8 mm, vias 0 -> 7
- net +1V8: track 0.00 -> 79.9 mm, vias 0 -> 8
- net +3V3: track 0.00 -> 72.3 mm, vias 0 -> 4
- net SIM7080G_PWR: track 0.00 -> 49.0 mm, vias 0 -> 4
- net Net-(D2-K): track 0.00 -> 43.3 mm, vias 0 -> 1
- net Net-(C7-Pad2): track 0.00 -> 42.7 mm, vias 0 -> 3
- net SIM_RST: track 0.00 -> 42.2 mm, vias 0 -> 5
- net Net-(D1-K): track 0.00 -> 39.3 mm, vias 0 -> 3
- net SIM_DATA: track 0.00 -> 34.7 mm, vias 0 -> 2
- net Net-(J4-Pad1): track 0.00 -> 33.9 mm, vias 0 -> 2
- net STATUS: track 0.00 -> 32.9 mm, vias 0 -> 3
- net SIM7080G_SDA: track 0.00 -> 31.6 mm, vias 0 -> 2
- net GNSS_ANT: track 0.00 -> 29.9 mm, vias 0 -> 2
- net Net-(JP1-B): track 0.00 -> 29.8 mm, vias 0 -> 1
- net SIM_CLK: track 0.00 -> 29.6 mm, vias 0 -> 2
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
Commit message: Route PCB
Signed-off-by: JeffMboya <jangina.mboya@gmail.com>
Routing:
- net SIM7080G_SCL: track 0.00 -> 74.2 mm, vias 0 -> 3
- net GND: track 185.8 -> 217.1 mm, vias 7 -> 13
- net NETLIGHT: track 0.00 -> 12.2 mm, vias 0 -> 3
- net +3V3: track 72.3 -> 80.2 mm, vias 4 -> 5
- net SIM_VDD: track 29.3 -> 37.1 mm, vias 5 -> 6
- net +1V8: track 79.9 -> 83.7 mm, vias 8 -> 11
- net SIM_RST: track 42.2 -> 42.9 mm

Commit message: Route PCB
Signed-off-by: JeffMboya <jangina.mboya@gmail.com>
Routing:
- net SIM7080G_TXD: track 0.00 -> 20.4 mm, vias 0 -> 4
- net Net-(Q1-B): track 1.60 -> 11.9 mm, vias 0 -> 2
- net SIM_VDD: track 37.1 -> 42.6 mm
- net GND: track 217.1 -> 220.7 mm, vias 13 -> 15

Commit message: Route PCB
Signed-off-by: JeffMboya <jangina.mboya@gmail.com>
Routing:
- net SIM_DATA: track 34.7 -> 15.5 mm, vias 2 -> 1
- net SIM7080G_PWR: track 49.0 -> 36.6 mm, vias 4 -> 3
- net +1V8: track 83.7 -> 87.9 mm, vias 11 -> 15
- net RF_ANT: track 20.8 -> 23.6 mm, vias 1 -> 2
- net GND: track 220.7 -> 218.6 mm, vias 15 -> 17
- net NETLIGHT: track 12.2 -> 11.4 mm, vias 3 -> 2
- net PWR_KEY: track 22.5 -> 23.0 mm, vias 1 -> 2
- net STATUS: track 32.9 -> 33.3 mm, vias 3 -> 4
- net Net-(C7-Pad2): track 42.7 -> 43.0 mm, vias 3 -> 4
- net +3V3: track 80.2 -> 80.1 mm, vias 5 -> 8
- net Net-(D2-K): vias 1 -> 2
- net SIM_VDD: vias 6 -> 7
- net Net-(JP1-B): vias 1 -> 2
- net Net-(JP1-A): vias 2 -> 3
- net GNSS_ANT: vias 2 -> 3

Commit message: Add power and ground planes
Signed-off-by: JeffMboya <jangina.mboya@gmail.com>
Routing:
- net SIM_DATA: track 15.5 -> 38.6 mm, vias 1 -> 3
- net SIM7080G_PWR: track 36.6 -> 15.8 mm
- net GND: track 218.6 -> 213.1 mm
- added copper zone on F.Cu, net +1V8
- added copper zone on In1.Cu, net +1V8
- added copper zone on F.Cu, net +3V3
- added copper zone on In2.Cu, net +3V3
- added copper zone on B.Cu, net GND
- added copper zone on F.Cu, net GND
Changed lines of the file:
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@@
 	)
 	(segment
-		(start 102 88.6375)
-		(end 101.4 89.2375)
+		(start 85.35 71.008578)
+		(end 86.358578 70)
 		(width 0.2)
 		(layer "F.Cu")
@@
 	)
 	(segment
-		(start 85.35 71.008578)
-		(end 86.358578 70)
+		(start 102.3 88.9)
+		(end 102.4875 89.0875)
 		(width 0.2)
 		(layer "F.Cu")
@@
 	)
 	(segment
-		(start 101.0125 89.2375)
-		(end 100.9875 89.2625)
-		(width 0.2)
-		(layer "F.Cu")
-		(net 1)
-	)
-	(segment
-		(start 100.9875 89.2625)
-		(end 100.9875 90.2625)
-		(width 0.2)
-		(layer "F.Cu")
-		(net 1)
-	)
-	(segment
 		(start 91.663136 86.650001)
 		(end 91.58 86.566865)
@@
 	)
 	(segment
-		(start 102.4875 89.2625)
-		(end 102.4625 89.2375)
-		(width 0.2)
-		(layer "F.Cu")
-		(net 1)
-	)
-	(segment
 		(start 88.8 59)
 		(end 88.8 59.248528)
@@
 	)
 	(segment
-		(start 102.4625 89.2375)
-		(end 101.4 89.2375)
-		(width 0.2)
-		(layer "F.Cu")
-		(net 1)
-	)
-	(segment
 		(start 86.6 59.8)
 		(end 86.7 59.7)
@@
 	)
 	(segment
-		(start 102.4875 90.2625)
-		(end 102.4875 89.2625)
-		(width 0.2)
-		(layer "F.Cu")
-		(net 1)
-	)
-	(segment
 		(start 89.8 89.1)
 		(end 89.9875 89.2875)
@@
 	)
 	(segment
+		(start 102.3 88.8)
+		(end 102.3 88.9)
+		(width 0.2)
+		(layer "F.Cu")
+		(net 1)
+	)
+	(segment
 		(start 94.1 86.5)
 		(end 94.1 87.160974)
@@
 	)
 	(segment
+		(start 100.9875 89.2625)
+		(end 101.45 88.8)
+		(width 0.2)
+		(layer "F.Cu")
+		(net 1)
+	)
+	(segment
 		(start 99.8875 56.3125)
 		(end 99.8875 55.7125)
@@
 	)
 	(segment
+		(start 102.4875 89.0875)
+		(end 102.4875 90.2625)
+		(width 0.2)
+		(layer "F.Cu")
+		(net 1)
+	)
+	(segment
 		(start 96.4 71.5)
 		(end 96.1 71.2)
@@
 	)
 	(segment
-		(start 96.8 87.3)
-		(end 97.2625 87.7625)
+		(start 83.3 84.8)
+		(end 84.8 84.8)
 		(width 0.2)
 		(layer "F.Cu")
@@
 	)
 	(segment
-		(start 83.3 84.8)
-		(end 84.8 84.8)
+		(start 100.9875 90.2625)
+		(end 100.9875 89.2625)
 		(width 0.2)
 		(layer "F.Cu")
@@
 	)
 	(segment
-		(start 94.239026 87.3)
-		(end 96.8 87.3)
-		(width 0.2)
-		(layer "F.Cu")
-		(net 1)
-	)
-	(segment
 		(start 85.65 89.1)
 		(end 86.5 89.1)
@@
 	)
 	(segment
+		(start 101.45 88.8)
+		(end 102.3 88.8)
+		(width 0.2)
+		(layer "F.Cu")
+		(net 1)
+	)
+	(segment
 		(start 94.6 72.6)
 		(end 93.2 71.2)
@@
 	)
 	(segment
-		(start 97.2625 87.7625)
-		(end 97.2625 88.811028)
-		(width 0.2)
-		(layer "F.Cu")
-		(net 1)
-	)
-	(segment
-		(start 101.4 89.2375)
-		(end 101.0125 89.2375)
-		(width 0.2)
-		(layer "F.Cu")
-		(net 1)
-	)
-	(segment
 		(start 92.1 76.9)
 		(end 91.4 77.6)
@@
 	)
 	(segment
-		(start 102 87.7)
-		(end 102 88.6375)
-		(width 0.2)
-		(layer "F.Cu")
-		(net 1)
-	)
-	(segment
 		(start 90.3 88.6)
 		(end 90.3 87.996948)
@@
 	)
 	(via
+		(at 98.475 79.75345)
+		(size 0.6)
+		(drill 0.3)
+		(layers "F.Cu" "B.Cu")
+		(net 10)
+	)
+	(via
 		(at 95.275735 58.875735)
 		(size 0.6)
@@
 		(net 10)
 	)
+	(via
+		(at 91.784864 75.364684)
+		(size 0.6)
+		(drill 0.3)
+		(layers "F.Cu" "B.Cu")
+		(net 10)
+	)
+	(segment
+		(start 98.475 79.025)
+		(end 98.475 79.75345)
+		(width 0.2)
+		(layer "In2.Cu")
+		(net 10)
+	)
+	(segment
+		(start 91.784864 75.364684)
+		(end 92.149548 75)
+		(width 0.2)
+		(layer "In2.Cu")
+		(net 10)
+	)
+	(segment
+		(start 99.9 76.700001)
+		(end 99.9 77.6)
+		(width 0.2)
+		(layer "In2.Cu")
+		(net 10)
+	)
+	(segment
+		(start 99.9 77.6)
+		(end 98.475 79.025)
+		(width 0.2)
+		(layer "In2.Cu")
+		(net 10)
+	)
+	(segment
+		(start 98.199999 75)
+		(end 99.9 76.700001)
+		(width 0.2)
+		(layer "In2.Cu")
+		(net 10)
+	)
+	(segment
+		(start 92.149548 75)
+		(end 98.199999 75)
+		(width 0.2)
+		(layer "In2.Cu")
+		(net 10)
+	)
 	(segment
 		(start 88.65147 65.5)
-		(end 95.275735 58.875735)
+		(end 88.775735 65.375735)
+		(width 0.2)
+		(layer "B.Cu")
+		(net 10)
+	)
+	(segment
+		(start 88.775735 65.375735)
+		(end 91.784864 68.384864)
+		(width 0.2)
+		(layer "B.Cu")
+		(net 10)
+	)
+	(segment
+		(start 91.784864 68.384864)
+		(end 91.784864 75.364684)
 		(width 0.2)
 		(layer "B.Cu")
@@
 	)
 	(segment
-		(start 98.3 78.934314)
+		(start 98.475 79.75345)
+		(end 98.3 79.92845)
+		(width 0.2)
+		(layer "B.Cu")
+		(net 10)
+	)
+	(segment
+		(start 98.3 79.92845)
 		(end 98.3 83.8)
 		(width 0.2)
@@
 	)
 	(segment
+		(start 88.775735 65.375735)
+		(end 95.275735 58.875735)
+		(width 0.2)
+		(layer "B.Cu")
+		(net 10)
+	)
+	(segment
 		(start 87.65 65.5)
 		(end 88.3 65.5)
@@
 	)
 	(segment
-		(start 88.525 66.725)
-		(end 86.764215 66.725)
-		(width 0.2)
-		(layer "B.Cu")
-		(net 70)
-	)
-	(segment
-		(start 88.525 70.63)
-		(end 88.525 66.725)
-		(width 0.2)
-		(layer "B.Cu")
-		(net 70)
-	)
-	(segment
 		(start 88.348529 55.724999)
 		(end 88.348529 56.802942)
@@
 	)
 	(segment
-		(start 86.764215 66.725)
-		(end 86.575 66.914215)
-		(width 0.2)
-		(layer "B.Cu")
-		(net 70)
-	)
-	(segment
-		(start 88.306627 87.362088)
-		(end 88.2 87.255461)
+		(start 88.525 66.725)
+		(end 86.764215 66.725)
 		(width 0.2)
 		(layer "B.Cu")
@@
 	)
 	(segment
-		(start 88.2 70.955)
-		(end 88.525 70.63)
-		(width 0.2)
-		(layer "B.Cu")
-		(net 70)
-	)
-	(segment
 		(start 88.348529 56.802942)
 		(end 87.2 57.951471)
@@
 	)
 	(segment
-		(start 88.2 87.255461)
-		(end 88.2 70.955)
-		(width 0.2)
-		(layer "B.Cu")
-		(net 70)
-	)
-	(segment
-		(start 86.575 66.914215)
+		(start 86.764215 66.725)
 		(end 86.591462 66.897753)
 		(width 0.2)
@@
 		(net 118)
 	)
+	(zone
+		(net 1)
+		(net_name "GND")
+		(layer "F.Cu")
+		(hatch edge 0.5)
+		(connect_pads
+			(clearance 0.5)
+		)
+		(min_thickness 0.25)
+		(filled_areas_thickness no)
+		(fill yes
+			(thermal_gap 0.5)
+			(thermal_bridge_width 0.5)
+		)
+		(polygon
+			(pts
+				(xy 79.8 47) (xy 105.5 46.7) (xy 106.4 94.1) (xy 79.5 93.4)
+			)
+		)
+	)
+	(zone
+		(net 5)
+		(net_name "+1V8")
+		(layers "F.Cu" "In1.Cu")
+		(hatch edge 0.5)
+		(priority 2)
+		(connect_pads
+			(clearance 0.5)
+		)
+		(min_thickness 0.25)
+		(filled_areas_thickness no)
+		(fill yes
+			(thermal_gap 0.5)
+			(thermal_bridge_width 0.5)
+		)
+		(polygon
+			(pts
+				(xy 76.8 44.3) (xy 107.6 44) (xy 109 96.4) (xy 77 96.5)
+			)
+		)
+	)
+	(zone
+		(net 18)
+		(net_name "+3V3")
+		(layers "F.Cu" "In2.Cu")
+		(hatch edge 0.5)
+		(priority 3)
+		(connect_pads
+			(clearance 0.5)
+		)
+		(min_thickness 0.25)
+		(filled_areas_thickness no)
+		(fill yes
+			(thermal_gap 0.5)
+			(thermal_bridge_width 0.5)
+		)
+		(polygon
+			(pts
+				(xy 75.3 42.4) (xy 108.5 41.9) (xy 111 98.1) (xy 74.4 98.3) (xy 75.4 42.4)
+			)
+		)
+	)
+	(zone
+		(net 1)
+		(net_name "GND")
+		(layers "F&B.Cu")
+		(hatch edge 0.5)
+		(priority 1)
+		(connect_pads
+			(clearance 0.5)
+		)
+		(min_thickness 0.25)
+		(filled_areas_thickness no)
+		(fill yes
+			(thermal_gap 0.5)
+			(thermal_bridge_width 0.5)
+		)
+		(polygon
+			(pts
+				(xy 78.4 46) (xy 106.5 45.3) (xy 107.7 94.9) (xy 78.2 95.5) (xy 78.6 46)
+			)
+		)
+	)
 )

Commit message: Route PCB
Signed-off-by: JeffMboya <jangina.mboya@gmail.com>
Parts:
- D3, J4, Q1: moved to B.Cu
- moved R15 30.8 mm to (83.3, 85.4), turned to -90 degrees
- moved C7 30.7 mm to (99.4, 79.9), turned to -90 degrees
- moved R7 23.1 mm to (83.1, 75.8), turned to 90 degrees
- moved R8 16.2 mm to (83.1, 63.4), turned to -90 degrees
- moved R10 16.0 mm to (103.3, 63.0), turned to 90 degrees
- moved C10 14.7 mm to (103.3, 67.5)
- moved C2 14.7 mm to (83.1, 67.9)
- moved R1 13.8 mm to (82.9, 71.8), turned to -90 degrees
- moved R5 13.3 mm to (103.3, 72.5)
- moved Q1 12.0 mm to (92.8, 75.4), turned to 90 degrees
- moved R14 11.8 mm to (87.3, 53.9)
- moved R12 11.6 mm to (83.2, 59.2), turned to 90 degrees
- moved J4 10.5 mm to (89.4, 75.4)
- moved C11 8.94 mm to (90.3, 85.3)
- moved D3 7.65 mm to (97.2, 75.7)
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Routing:
- net Net-(C7-Pad2): track 43.0 -> 7.51 mm, vias 4 -> 0
- net Net-(J4-Pad1): track 33.9 -> 5.15 mm, vias 2 -> 1
- net Net-(Q3-B): track 12.9 -> 40.3 mm, vias 0 -> 4
- net GNSS_ANT: track 29.9 -> 5.83 mm, vias 3 -> 0
- net SIM7080G_SCL: track 74.2 -> 50.6 mm, vias 3 -> 4
- net +3V3: track 80.1 -> 103.2 mm, vias 8 -> 13
- net Net-(D1-K): track 39.3 -> 20.0 mm
- net Net-(D4-A): track 10.8 -> 29.6 mm, vias 0 -> 2
- net RF_ANT: track 23.6 -> 5.32 mm
- net PWR_KEY: track 23.0 -> 39.0 mm
- net +1V8: track 87.9 -> 73.1 mm, vias 15 -> 10
- net SIM_CLK: track 29.6 -> 44.2 mm, vias 2 -> 4
- net SIM7080G_TXD: track 20.4 -> 8.10 mm, vias 4 -> 2
- net SIM_RST: track 42.9 -> 31.2 mm, vias 5 -> 4
- net Net-(D2-K): track 43.3 -> 33.0 mm
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- removed copper zone on F.Cu, net +1V8
- removed copper zone on In1.Cu, net +1V8
- removed copper zone on F.Cu, net +3V3
- removed copper zone on In2.Cu, net +3V3
- removed copper zone on B.Cu, net GND
- removed copper zone on F.Cu, net GND

Commit message: Add ground and power planes
Signed-off-by: JeffMboya <jangina.mboya@gmail.com>
Routing:
- net (no net): track 1.10 -> 7.34 mm
- added copper zone on In2.Cu, net +1V8
- added copper zone on In1.Cu, net +3V3
- added copper zone on B.Cu, net GND
- added copper zone on F.Cu, net GND
Changed lines of the file:
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@@
 	)
 	(segment
+		(start 86.931583 66.906436)
+		(end 86.088019 67.75)
+		(width 0)
+		(layer "F.Cu")
+		(net 0)
+	)
+	(segment
+		(start 84.742893 66.65)
+		(end 85.35 66.65)
+		(width 0)
+		(layer "F.Cu")
+		(net 0)
+	)
+	(segment
+		(start 84.35 67.042893)
+		(end 84.742893 66.65)
+		(width 0)
+		(layer "F.Cu")
+		(net 0)
+	)
+	(segment
+		(start 86.2 65.7)
+		(end 86.931583 66.431583)
+		(width 0)
+		(layer "F.Cu")
+		(net 0)
+	)
+	(segment
+		(start 85.35 67.75)
+		(end 85.4 67.75)
+		(width 0)
+		(layer "F.Cu")
+		(net 0)
+	)
+	(segment
+		(start 84.35 67.457107)
+		(end 84.35 67.042893)
+		(width 0)
+		(layer "F.Cu")
+		(net 0)
+	)
+	(segment
 		(start 85.35 69.45)
 		(end 85.35 68.35)
@@
 	)
 	(segment
+		(start 86.931583 66.431583)
+		(end 86.931583 66.906436)
+		(width 0)
+		(layer "F.Cu")
+		(net 0)
+	)
+	(segment
+		(start 85.4 67.75)
+		(end 84.642893 67.75)
+		(width 0)
+		(layer "F.Cu")
+		(net 0)
+	)
+	(segment
+		(start 84.642893 67.75)
+		(end 84.35 67.457107)
+		(width 0)
+		(layer "F.Cu")
+		(net 0)
+	)
+	(segment
+		(start 86.088019 67.75)
+		(end 85.35 67.75)
+		(width 0)
+		(layer "F.Cu")
+		(net 0)
+	)
+	(segment
 		(start 89.725 57.675)
 		(end 90.375 57.675)
@@
 		(net 118)
 	)
+	(zone
+		(net 1)
+		(net_name "GND")
+		(layers "F&B.Cu")
+		(hatch edge 0.5)
+		(connect_pads
+			(clearance 0.5)
+		)
+		(min_thickness 0.25)
+		(filled_areas_thickness no)
+		(fill yes
+			(thermal_gap 0.5)
+			(thermal_bridge_width 0.5)
+		)
+		(polygon
+			(pts
+				(xy 80.2 45.7) (xy 107.4 45.4) (xy 107.3 93.6) (xy 80.1 94.3) (xy 80.2 45.7)
+			)
+		)
+	)
+	(zone
+		(net 18)
+		(net_name "+3V3")
+		(layer "In1.Cu")
+		(hatch edge 0.5)
+		(priority 1)
+		(connect_pads
+			(clearance 0.5)
+		)
+		(min_thickness 0.25)
+		(filled_areas_thickness no)
+		(fill yes
+			(thermal_gap 0.5)
+			(thermal_bridge_width 0.5)
+		)
+		(polygon
+			(pts
+				(xy 78.8 43.7) (xy 109 44.2) (xy 108.8 95.6) (xy 78.4 95.9)
+			)
+		)
+	)
+	(zone
+		(net 5)
+		(net_name "+1V8")
+		(layer "In2.Cu")
+		(hatch edge 0.5)
+		(priority 2)
+		(connect_pads
+			(clearance 0.5)
+		)
+		(min_thickness 0.25)
+		(filled_areas_thickness no)
+		(fill yes
+			(thermal_gap 0.5)
+			(thermal_bridge_width 0.5)
+		)
+		(polygon
+			(pts
+				(xy 77.6 42.6) (xy 110.9 42.8) (xy 110 98.1) (xy 76.3 97.9) (xy 77.5 42.7)
+			)
+		)
+	)
 )
