File: modules/compute/output.kicad_pcb (KiCad board)
At the start: 2 copper layers, 86 x 30 mm, 80 parts, among them J1 Bus_M.2_Socket_E, J2 Conn_ARM_SWD_TagConnect_TC203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, SW1 SW_Push, U1 ESP32-C3-MINI-1U-H4

Commit message: Fix right angled tracks
Signed-off-by: JeffMboya <jangina.mboya@gmail.com>
Routing:
- net Board_0-GND: track 162.9 -> 158.3 mm
- net Board_2-GND: track 162.9 -> 162.2 mm
- net Board_1-GND: track 162.9 -> 162.4 mm
