File: modules/sim7080G/peripherals.kicad_sch (KiCad schematic)
At the start: 38 parts, among them J3 GNSS Antenna, J4 RF Antenna, J5 NSIM-5-B, Q1 SS8050, Q2 SS8050, Q3 SS8050, U2 SIM7080G, U3 TXB0108RGY

Commit message: fix: remodify board to be a baseboard
Signed-off-by: Rodney Osodo <socials@rodneyosodo.com>
Parts:
- J3, J4: footprint CONUFL001_SMD_T:CONN1_CONUFL_TEC -> CONUFL001:CONN1_CONUFL_TEC
Changed lines of the file:
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@@
 			)
 		)
-		(property "Footprint" "CONUFL001_SMD_T:CONN1_CONUFL_TEC"
+		(property "Footprint" "CONUFL001:CONN1_CONUFL_TEC"
 			(at 361.95 34.29 0)
 			(effects
@@
 			)
 		)
-		(property "Footprint" "CONUFL001_SMD_T:CONN1_CONUFL_TEC"
+		(property "Footprint" "CONUFL001:CONN1_CONUFL_TEC"
 			(at 363.22 69.85 0)
 			(effects
