File: modules/s0/wmbus.kicad_sch (KiCad schematic)
At the start: 2 parts, among them U6 RC-S2LP-868

Commit message: chore: add production files
Changed lines of the file:
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@@
-		)
-	)
-	(rectangle
-		(start 66.04 26.67)
-		(end 213.36 146.05)
-		(stroke
-			(width 1)
-			(type default)
-			(color 89 10 255 1)
-		)
-		(fill
-			(type none)
 		)
 	)

Commit message: chore:Modify BOM in production
Connections:
- no-connect marks 0 -> 4
Changed lines of the file:
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@@
 		(comment 2 "Approved By: Jones Kisaka")
+	)
+	(no_connect
+		(at 139.7 73.66)
+	)
+	(no_connect
+		(at 139.7 76.2)
+	)
+	(no_connect
+		(at 139.7 81.28)
+	)
+	(no_connect
+		(at 139.7 78.74)
 	)
 	(wire

Commit message: Modified Schematics and BOM
Parts:
- renumbered C19 to C18, U6 to U8
Changed lines of the file:
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@@
 		(dnp no)
 		(fields_autoplaced yes)
-		(property "Reference" "#PWR02"
+		(property "Reference" "#PWR062"
 			(at 144.78 93.98 0)
 			(effects
@@
 			(project "s0"
 				(path "/9e4c0f80-14bc-451b-8b05-b2f0d1a90e15/3bbb84ad-503a-4b2d-9543-6ed81c985ce9"
-					(reference "#PWR02")
+					(reference "#PWR062")
 					(unit 1)
 				)
@@
 		(dnp no)
 		(fields_autoplaced yes)
-		(property "Reference" "#PWR057"
+		(property "Reference" "#PWR063"
 			(at 165.1 67.31 0)
 			(effects
@@
 			(project "s0"
 				(path "/9e4c0f80-14bc-451b-8b05-b2f0d1a90e15/3bbb84ad-503a-4b2d-9543-6ed81c985ce9"
-					(reference "#PWR057")
+					(reference "#PWR063")
 					(unit 1)
 				)
@@
 		(dnp no)
 		(fields_autoplaced yes)
-		(property "Reference" "U6"
+		(property "Reference" "U8"
 			(at 124.46 55.88 0)
 			(effects
@@
 			(project ""
 				(path "/9e4c0f80-14bc-451b-8b05-b2f0d1a90e15/3bbb84ad-503a-4b2d-9543-6ed81c985ce9"
-					(reference "U6")
+					(reference "U8")
 					(unit 1)
 				)
@@
 		(dnp no)
 		(fields_autoplaced yes)
-		(property "Reference" "#PWR056"
+		(property "Reference" "#PWR064"
 			(at 165.1 90.17 0)
 			(effects
@@
 			(project "s0"
 				(path "/9e4c0f80-14bc-451b-8b05-b2f0d1a90e15/3bbb84ad-503a-4b2d-9543-6ed81c985ce9"
-					(reference "#PWR056")
+					(reference "#PWR064")
 					(unit 1)
 				)
@@
 		(dnp no)
 		(fields_autoplaced yes)
-		(property "Reference" "#PWR01"
+		(property "Reference" "#PWR061"
 			(at 143.51 64.77 0)
 			(effects
@@
 			(project "s0"
 				(path "/9e4c0f80-14bc-451b-8b05-b2f0d1a90e15/3bbb84ad-503a-4b2d-9543-6ed81c985ce9"
-					(reference "#PWR01")
+					(reference "#PWR061")
 					(unit 1)
 				)
@@
 		(dnp no)
 		(fields_autoplaced yes)
-		(property "Reference" "C19"
+		(property "Reference" "C18"
 			(at 168.91 73.6599 0)
 			(effects
@@
 			)
 		)
-		(property "Description" "Unpolarized capacitor"
+		(property "Description" "16V 100nF X7R ±10% 0402 Multilayer Ceramic Capacitors MLCC - SMD/SMT ROHS"
 			(at 165.1 74.93 0)
 			(effects
@@
 			(project "s0"
 				(path "/9e4c0f80-14bc-451b-8b05-b2f0d1a90e15/3bbb84ad-503a-4b2d-9543-6ed81c985ce9"
-					(reference "C19")
+					(reference "C18")
 					(unit 1)
 				)

Commit message: chore: route the board with changes
Parts:
- U8: footprint Module:XCVR_RC-S2LP-868 -> modules:XCVR_RC-S2LP-868
Changed lines of the file:
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@@
 			)
 		)
-		(property "Footprint" "Module:XCVR_RC-S2LP-868"
+		(property "Footprint" "modules:XCVR_RC-S2LP-868"
 			(at 124.46 76.2 0)
 			(effects
