File: modules/s0-base-board/s0-base-board.kicad_pcb (KiCad board)
At the start: 2 copper layers, 54.6 x 86.4 mm, 81 parts, among them J2 Screw_Terminal_01x02, J3 BAT_JST_01x02, J4 RJ45_Bel_SI-60062-F JLC, J5 Conn_02x23_Odd_Even, J6 Conn_02x23_Odd_Even, Q1 PMOS, U1 MCP73831-2-OT, U2 XL1509-5.0, U3 LM2575S-3.3(UMW), U4 W5500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

Commit message: Reviewed Changes made
Parts:
- added F1: Fuse, Module:FUSC3115X66N, F.Cu at (187.0, 111.5)
- added L5: Ferrite Bead, Module:BEADC3216X130N, F.Cu at (178.5, 125.0)
- added Q2: 2N5401, Module:SOT95P230X117-3N, F.Cu at (180.5, 68.0)
- added Q3: IRF4905STRLPBF, Module:TRANS_IRF3205S, F.Cu at (171.0, 67.5)
- added R22: 1k, Resistor_SMD:R_0402_1005Metric, F.Cu at (163.0, 60.0)
- added R3: 1k, Resistor_SMD:R_0402_1005Metric, F.Cu at (174.0, 53.5)
- moved C4 14.6 mm to (169.0, 79.0), turned to 180 degrees
- moved D6 8.28 mm to (174.0, 56.5), turned to 180 degrees
- moved L1 7.58 mm to (169.5, 85.5)
- moved D2 7.53 mm to (170.4, 94.0)
- moved C7 4.42 mm to (176.0, 120.0), turned to 90 degrees
- moved C6 4.20 mm to (180.0, 76.0)
- moved R20 4.12 mm to (178.0, 51.0)
- moved kibuzzard-67D30BB5 3.53 mm to (176.5, 46.5)
- moved R2 2.24 mm to (172.0, 54.0), turned to 0 degrees
- moved kibuzzard-67D30BA5 1.85 mm to (162.0, 48.0)
- moved J2 1.61 mm to (167.0, 48.0)
- moved U2 1.42 mm to (179.0, 80.1)
Connections:
- C5 pad 1: Net-(D3-K) -> Net-(U3-VIN)
- C7 pad 1: +3V3 -> Net-(U3-FB)
- D6 pad 1: VIN -> Net-(D6-K)
- L2 pad 2: +3V3 -> Net-(U3-FB)
- R2 pad 1: VIN -> Net-(D5-K)
- R2 pad 2: Net-(D5-K) -> Net-(D6-K)
- U3 pad 1: Net-(D3-K) -> Net-(U3-VIN)
- U3 pad 4: +3V3 -> Net-(U3-FB)
Routing:
- net Net-(U3-FB): track 0.00 -> 52.3 mm
- net Net-(D5-K): track 4.50 -> 55.1 mm, vias 0 -> 2
- net GND: track 421.8 -> 461.9 mm, vias 5 -> 11
- net Net-(Q2-C): track 0.00 -> 21.3 mm
- net Net-(D3-K): track 53.5 -> 33.6 mm
- net Net-(U3-VIN): track 0.00 -> 19.2 mm, vias 0 -> 2
- net Net-(Q2-B): track 0.00 -> 15.9 mm
- net VIN: track 27.0 -> 12.2 mm
- net LINKLED: track 64.0 -> 72.3 mm
- net +3V3: track 141.1 -> 134.6 mm, vias 5 -> 7
- net Net-(D6-K): track 0.00 -> 6.48 mm
- net +5V: track 119.1 -> 123.9 mm, vias 2 -> 4
- net Net-(D2-K): track 13.7 -> 17.6 mm
- net Net-(J4-PadL4): track 7.51 -> 4.60 mm
- net Net-(D5-A): track 7.59 -> 9.28 mm

Commit message: Reviewed Changes
Parts:
- added D7: LED, LED_SMD:LED_0603_1608Metric, F.Cu at (168.0, 123.5)
- added R23: 220, Resistor_SMD:R_0402_1005Metric, F.Cu at (167.8, 120.5)
- added TP1: TestPoint, TestPoint:TestPoint_Pad_D1.0mm, F.Cu at (208.5, 123.0)
- added TP2: TestPoint, TestPoint:TestPoint_Pad_D1.0mm, F.Cu at (206.0, 123.0)
- added TP3: TestPoint, TestPoint:TestPoint_Pad_D1.0mm, F.Cu at (211.0, 123.0)
- added TP4: TestPoint, TestPoint:TestPoint_Pad_D1.0mm, F.Cu at (203.5, 123.0)
- added kibuzzard-67ED70B8: G***, kibuzzard-67ED70B8, F.Cu at (203.5, 125.5)
- added kibuzzard-67ED70E0: G***, kibuzzard-67ED70E0, F.Cu at (206.0, 125.5)
- added kibuzzard-67ED70ED: G***, kibuzzard-67ED70ED, F.Cu at (168.0, 125.5)
- added kibuzzard-67ED70ED: G***, kibuzzard-67ED70ED, F.Cu at (208.5, 125.5)
- added kibuzzard-67ED70F9: G***, kibuzzard-67ED70F9, F.Cu at (211.0, 125.5)
Routing:
- net +3V3: track 134.6 -> 180.4 mm
- net +5V: track 123.9 -> 163.5 mm, vias 4 -> 6
- net Net-(D3-K): track 33.6 -> 55.9 mm, vias 2 -> 3
- net GND: track 461.9 -> 475.2 mm
- net Net-(D7-K): track 0.00 -> 3.03 mm

Commit message: Reviewed Changes
Parts:
- removed the kibuzzard-67ED70ED at (168.0, 125.5)
- added kibuzzard-67ED74E9: G***, kibuzzard-67ED74E9, F.Cu at (168.0, 125.5)

Commit message: fix(silkscreen): Add logo and website name
Parts:
- moved G*** 2.47 mm to (184.9, 80.1)
Other:
- board text added: "."
- board text added: "Base Board"
- board text added: "S0-BB"
- board text added: "www.absmach.eu"

Commit message: style: add new aligned logo
Parts:
- moved G*** 20.3 mm to (185.9, 100.3)
Other:
- board text removed: "."
- board text removed: "Base Board"
- board text removed: "S0-BB"
- board text removed: "www.absmach.eu"
