File: modules/s0-base-board/mbus.kicad_sch (KiCad schematic)
At the start: 8 parts, among them J1 Screw_Terminal_01x02, J7 METER-BUS TRANSCEIVER

Commit message: feat(base-board): route and add wirembus support
Signed-off-by: Rodney Osodo <socials@rodneyosodo.com>
Other:
- company: (none) -> Abstract Machines
- title: (none) -> S0 Base Board
Changed lines of the file:
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@@
 	(generator_version "8.0")
 	(paper "A4")
+	(title_block
+		(title "S0 Base Board")
+		(date "2025-02-26")
+		(rev "v0.1.0")
+		(company "Abstract Machines")
+		(comment 1 "Deigned By: Rodney Osodo")
+		(comment 2 "Approved By: Jones Kisaka")
+	)
 	(junction
 		(at 133.35 55.88)
@@
 			)
 		)
+		(property "LCSC Part" ""
+			(at 49.53 63.5 0)
+			(effects
+				(font
+					(size 1.27 1.27)
+				)
+				(hide yes)
+			)
+		)
 		(pin "2"
 		)
@@
 		)
 		(property "JLCPCB" "C412252"
+			(at 63.5 69.85 0)
+			(effects
+				(font
+					(size 1.27 1.27)
+				)
+				(hide yes)
+			)
+		)
+		(property "LCSC Part" ""
 			(at 63.5 69.85 0)
 			(effects
@@
 			)
 		)
+		(property "LCSC Part" ""
+			(at 124.46 55.88 0)
+			(effects
+				(font
+					(size 1.27 1.27)
+				)
+				(hide yes)
+			)
+		)
 		(pin "2"
 		)
@@
 			)
 		)
+		(property "LCSC Part" ""
+			(at 177.8 63.5 0)
+			(effects
+				(font
+					(size 1.27 1.27)
+				)
+				(hide yes)
+			)
+		)
 		(pin "2"
 		)
@@
 			)
 		)
+		(property "LCSC Part" ""
+			(at 114.3 50.8 0)
+			(effects
+				(font
+					(size 1.27 1.27)
+				)
+				(hide yes)
+			)
+		)
 		(pin "2"
 		)
@@
 			)
 		)
+		(property "LCSC Part" ""
+			(at 77.47 50.8 0)
+			(effects
+				(font
+					(size 1.27 1.27)
+				)
+				(hide yes)
+			)
+		)
 		(pin "2"
 		)
@@
 		)
 		(property "JLCPCB" "C34958"
+			(at 93.98 58.42 0)
+			(effects
+				(font
+					(size 1.27 1.27)
+				)
+				(hide yes)
+			)
+		)
+		(property "LCSC Part" ""
 			(at 93.98 58.42 0)
 			(effects
@@
 			(at 66.04 58.42 0)
 			(effects
+				(font
+					(size 1.27 1.27)
+				)
+				(hide yes)
+			)
+		)
+		(property "LCSC Part" ""
+			(at 66.04 58.42 0)
+			(effects

Commit message: Pin Changes. Baseboard-S0 sync
Parts:
- R25, R26: footprint Resistor_SMD:R_0402_1005Metric -> Resistor_SMD:R_0603_1608Metric; JLCPCB C1111 -> C22962
Changed lines of the file:
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@@
 			)
 		)
-		(property "Footprint" "Resistor_SMD:R_0402_1005Metric"
+		(property "Footprint" "Resistor_SMD:R_0603_1608Metric"
 			(at 114.3 49.022 90)
 			(effects
@@
 			)
 		)
-		(property "JLCPCB" "C1111"
+		(property "JLCPCB" "C22962"
 			(at 114.3 50.8 0)
 			(effects
@@
 			)
 		)
-		(property "Footprint" "Resistor_SMD:R_0402_1005Metric"
+		(property "Footprint" "Resistor_SMD:R_0603_1608Metric"
 			(at 77.47 49.022 90)
 			(effects
@@
 			)
 		)
-		(property "JLCPCB" "C1111"
+		(property "JLCPCB" "C22962"
 			(at 77.47 50.8 0)
 			(effects
