File: s0/esp32-c6.kicad_sch (KiCad schematic)
At the start: 11 parts, among them J1 Conn_ARM_JTAG_SWD_10, SW1 SW_Push, SW2 SW_Push, U1 ESP32-C6-MINI-1/U

Commit message: feat: finish routing on S0
Parts:
- C1: JLCPCB (none) -> C45783
- C2: JLCPCB (none) -> C15850
- C3, C4: JLCPCB (none) -> C49678
- J1: JLCPCB (none) -> C2935953
- R1, R2, R3: JLCPCB (none) -> C17414
- SW1, SW2: JLCPCB (none) -> C720477
- U1: footprint PCM_Espressif:ESP32-C6-MINI-1 -> modules:XCVR_ESP32-C3-MINI-1U-N4; JLCPCB (none) -> C20627095
Changed lines of the file:
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@@
+			)
+		)
+		(property "JLCPCB" "C17414"
+			(at 116.84 35.56 0)
+			(effects
+				(font
+					(size 1.27 1.27)
+				)
+				(hide yes)
 			)
 		)
@@
 			)
 		)
+		(property "JLCPCB" "C15850"
+			(at 195.58 38.1 0)
+			(effects
+				(font
+					(size 1.27 1.27)
+				)
+				(hide yes)
+			)
+		)
 		(pin "2"
 		)
@@
 			)
 		)
+		(property "JLCPCB" "C45783"
+			(at 177.8 38.1 0)
+			(effects
+				(font
+					(size 1.27 1.27)
+				)
+				(hide yes)
+			)
+		)
 		(pin "2"
 		)
@@
 			)
 		)
+		(property "JLCPCB" "C2935953"
+			(at 58.42 158.75 0)
+			(effects
+				(font
+					(size 1.27 1.27)
+				)
+				(hide yes)
+			)
+		)
 		(pin "6"
 		)
@@
 			)
 		)
+		(property "JLCPCB" "C17414"
+			(at 25.4 38.1 0)
+			(effects
+				(font
+					(size 1.27 1.27)
+				)
+				(hide yes)
+			)
+		)
 		(pin "1"
 		)
@@
 			)
 		)
+		(property "JLCPCB" "C720477"
+			(at 25.4 55.88 90)
+			(effects
+				(font
+					(size 1.27 1.27)
+				)
+				(hide yes)
+			)
+		)
 		(pin "1"
 		)
@@
 			)
 		)
+		(property "JLCPCB" "C720477"
+			(at 66.04 55.88 90)
+			(effects
+				(font
+					(size 1.27 1.27)
+				)
+				(hide yes)
+			)
+		)
 		(pin "1"
 		)
@@
 			)
 		)
+		(property "JLCPCB" "C49678"
+			(at 39.37 55.88 0)
+			(effects
+				(font
+					(size 1.27 1.27)
+				)
+				(hide yes)
+			)
+		)
 		(pin "2"
 		)
@@
 			)
 		)
-		(property "Footprint" "PCM_Espressif:ESP32-C6-MINI-1"
+		(property "Footprint" "modules:XCVR_ESP32-C3-MINI-1U-N4"
 			(at 226.06 131.445 0)
 			(effects
@@
 			)
 		)
+		(property "JLCPCB" "C20627095"
+			(at 226.06 86.36 0)
+			(effects
+				(font
+					(size 1.27 1.27)
+				)
+				(hide yes)
+			)
+		)
 		(pin "27"
 		)
@@
 			)
 		)
+		(property "JLCPCB" "C49678"
+			(at 80.01 55.88 0)
+			(effects
+				(font
+					(size 1.27 1.27)
+				)
+				(hide yes)
+			)
+		)
 		(pin "2"
 		)
@@
 			(at 66.04 38.1 0)
 			(effects
+				(font
+					(size 1.27 1.27)
+				)
+				(hide yes)
+			)
+		)
+		(property "JLCPCB" "C17414"
+			(at 66.04 38.1 0)
+			(effects
