File: s0/power.kicad_sch (KiCad schematic)
At the start: 24 parts, among them J4 ESP32 USB, J5 SIM7080G USBC, J6 Conn_01x02, J7 Beagle P9, J8 Beagle P8, U6 AMS1117-3.3

Commit message: feat: finish routing on S0
Parts:
- added H1, H2, H3, H4: MountingHole_Pad, MountingHole:MountingHole_2.5mm_Pad, symbol Mechanical:MountingHole_Pad
- C19, C21: JLCPCB (none) -> C15850
- C20, C22: JLCPCB (none) -> C49678
- D10, D11, D6, D7, D8, D9: JLCPCB (none) -> C111566
- D12: JLCPCB (none) -> C6848499
- F1: footprint (none) -> Fuse:Fuse_1206_3216Metric_Pad1.42x1.75mm_HandSolder; JLCPCB (none) -> C3105
- FB1: footprint (none) -> Inductor_SMD:L_1206_3216Metric_Pad1.22x1.90mm_HandSolder; JLCPCB (none) -> C668306
- J4, J5: JLCPCB (none) -> C2765186
- J6: JLCPCB (none) -> C20079
- J7, J8: JLCPCB (none) -> C725895
- R18, R19, R20, R21: JLCPCB (none) -> C27834
- R22: JLCPCB (none) -> C17540
- U6: JLCPCB (none) -> C6186
Connections:
- net GND: now also H1.1, H2.1, H3.1, H4.1
