File: s0/sim7080G.kicad_sch (KiCad schematic)
At the start: 41 parts, among them J2 Conn_Coaxial, J3 Conn_Coaxial, Q1 NPN, Q2 NPN, Q3 NPN, U2 SIM7080G, U3 NANO SIM XG6P H1.35, U4 TXB0108RGY

Commit message: feat: finish routing on S0
Parts:
- C10, C11: JLCPCB (none) -> C15850
- C12, C16, C17, C5, C7, C8, C9: JLCPCB (none) -> C49678
- C13, C14, C15: JLCPCB (none) -> C1804
- C6: footprint Capacitor_SMD:C_0805_2012Metric -> Capacitor_SMD:C_1206_3216Metric; JLCPCB (none) -> C15008
- D1, D2: JLCPCB (none) -> C111566
- D3: JLCPCB (none) -> C2935146
- D4, D5: JLCPCB (none) -> C6848499
- J2, J3: JLCPCB (none) -> C88373
- Q1, Q2, Q3: JLCPCB (none) -> C2150
- R10, R11: JLCPCB (none) -> C17408
- R12, R13, R6: JLCPCB (none) -> C17673
- R14, R15: JLCPCB (none) -> C17713
- R4: JLCPCB (none) -> C17414
- R5, R7, R8: JLCPCB (none) -> C17561
- R9: value R -> 47K; JLCPCB (none) -> C17713
- U2: footprint SIM7080G:XCVR_SIM7080G -> modules:XCVR_SIM7080G; JLCPCB (none) -> C2943992
- U3: footprint easyeda2kicad:SIM-SMD_NANO-SIM-XG6P-H1.35 -> modules:SIM-SMD_NANO-SIM-XG6P-H1.35; JLCPCB (none) -> C77877
- U4: JLCPCB (none) -> C194701
