File: s0/wmbus.kicad_sch (KiCad schematic)
At the start: 4 parts, among them U5 RC-S2LP-868

Commit message: feat: finish routing on S0
Parts:
- C18: JLCPCB (none) -> C49678
- R16: JLCPCB (none) -> C17408
- R17: JLCPCB (none) -> C17414
- U5: footprint RC-S2LP-868:XCVR_RC-S2LP-868 -> modules:XCVR_RC-S2LP-868; JLCPCB (none) -> C37069913
Changed lines of the file:
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@@
 			)
 		)
-		(property "Footprint" "RC-S2LP-868:XCVR_RC-S2LP-868"
+		(property "Footprint" "modules:XCVR_RC-S2LP-868"
 			(at 138.43 88.9 0)
 			(effects
@@
 				)
 				(justify bottom)
+				(hide yes)
+			)
+		)
+		(property "JLCPCB" "C37069913"
+			(at 138.43 88.9 0)
+			(effects
+				(font
+					(size 1.27 1.27)
+				)
 				(hide yes)
 			)
@@
 			)
 		)
+		(property "JLCPCB" "C17408"
+			(at 85.09 81.28 90)
+			(effects
+				(font
+					(size 1.27 1.27)
+				)
+				(hide yes)
+			)
+		)
 		(pin "2"
 		)
@@
 			)
 		)
+		(property "JLCPCB" "C17414"
+			(at 93.98 90.17 0)
+			(effects
+				(font
+					(size 1.27 1.27)
+				)
+				(hide yes)
+			)
+		)
 		(pin "2"
 		)
@@
 			(at 173.99 81.28 0)
 			(effects
+				(font
+					(size 1.27 1.27)
+				)
+				(hide yes)
+			)
+		)
+		(property "JLCPCB" "C49678"
+			(at 173.99 81.28 0)
+			(effects
