File: s0/s0.kicad_pcb (KiCad board)
At the start: 4 copper layers, 54.6 x 86.3 mm, 87 parts, among them J1 Conn_ARM_JTAG_SWD_10, J2 Conn_Coaxial, J3 Conn_Coaxial, J4 ESP32 USB, J5 SIM7080G USBC, J6 Conn_01x02, J7 Beagle P9, J8 Beagle P8, Q1 NPN, Q2 NPN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

Commit message: NOISSUE - S0 to A0 migration (#23)
Parts:
- moved G2 1.58 mm to (69.7, 107.5)
