File: a0/sim7080G.kicad_sch (KiCad schematic)
At the start: 41 parts, among them J2 Conn_Coaxial, J3 Conn_Coaxial, Q1 NPN, Q2 NPN, Q3 NPN, U2 SIM7080G, U3 NANO SIM XG6P H1.35, U4 TXB0108RGY

Commit message: update A0
Signed-off-by: Rodney Osodo <socials@rodneyosodo.com>
Connections:
- net SCL: no longer names the net of U4.12 (B8)
- net SDA: no longer names the net of U4.13 (B7)
- net SIM7080G_D+: no longer names the net of U2.25 (USB_DP)
- net SIM7080G_D-: no longer names the net of U2.26 (USB_DM)
- net SIM_SCL: no longer names the net of U2.65 (I2C_SCL)
- net SIM_SCL: no longer U4.9 (A8)
- net SIM_SDA: no longer names the net of U2.64 (I2C_SDA)
- net SIM_SDA: no longer U4.8 (A7)
- no-connect marks 22 -> 31
Other:
- note added: "ANTENNAE"
- note added: "DECOUPLING CAPS"
- note added: "NETLIGHT CTRL"
- note added: "POWER CTRL"
- note added: "SIM CARD"
- note added: "SIM7080G"
- note added: "STATUS CTRL"
- note added: "VOLTAGE CONVERTER"
- company: (none) -> Abstract Machines
- title: (none) -> A0
- moved on the sheet: C10, C11, C12, C13, C14, C15, C16, C17, C5, C6, C7, C8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
