File: a0/wmbus.kicad_sch (KiCad schematic)
At the start: 4 parts, among them U5 RC-S2LP-868

Commit message: update A0
Signed-off-by: Rodney Osodo <socials@rodneyosodo.com>
Other:
- note added: "WMBUS"
- company: (none) -> Abstract Machines
- title: (none) -> A0
Changed lines of the file:
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@@
 	(generator_version "9.0")
 	(paper "A4")
+	(title_block
+		(title "A0")
+		(date "2026-07-03")
+		(rev "v0.4.0")
+		(company "Abstract Machines")
+		(comment 1 "Designed By: Osodo Rodney")
+		(comment 2 "Approved By: Jones Kisaka")
+		(comment 3 "Approved By: Jeff Mboya")
+	)
 	(text "Datasheet: https://www.tme.eu/Document/670e39e2c98cd03151602fa1ab7255b3/RC-S2LP-868.pdf"
 		(exclude_from_sim no)
@@
 		)
 	)
+	(text "WMBUS"
+		(exclude_from_sim no)
+		(at 119.888 50.546 0)
+		(effects
+			(font
+				(size 5 5)
+				(thickness 1)
+				(bold yes)
+			)
+			(justify left bottom)
+		)
+	)
