File: modules/sim7080g/sim7080g.kicad_pcb (KiCad board)
At the start: 4 copper layers, 25.4 x 57.2 mm, 57 parts, among them J1 Conn_Coaxial, J2 Conn_01x08, J3 Conn_01x08, J4 Conn_Coaxial, Q1 NPN, Q2 NPN, Q3 NPN, U1 TXB0108RGY, U2 SIM7080G, U3 NANO SIM XG6P H1.35

Commit message: cross check sim7080G module is ready for fabrication
Signed-off-by: Rodney Osodo <socials@rodneyosodo.com>
Routing:
- net GND: track 6.69 -> 64.6 mm, vias 51 -> 87
- net SIM7080G_TX: track 27.5 -> 18.9 mm, vias 3 -> 2
- net +3V3: track 88.0 -> 79.6 mm, vias 8 -> 9
- net Net-(JP2-A): track 5.04 -> 12.5 mm, vias 1 -> 2
- net SIM_DATA: track 18.8 -> 26.1 mm, vias 6 -> 5
- net SIM_CLK: track 22.6 -> 16.4 mm, vias 6 -> 3
- net PWRKEY: track 22.6 -> 28.7 mm, vias 4 -> 3
- net SIM7080G_RING: track 21.0 -> 26.7 mm, vias 3 -> 2
- net SIM_VDD: track 31.9 -> 27.4 mm
- net SIM_TX: track 22.9 -> 27.1 mm
- net +1V8: track 34.4 -> 38.1 mm, vias 6 -> 5
- net RF_ANT: track 13.0 -> 16.5 mm, vias 0 -> 1
- net Net-(U3-I/O): track 5.23 -> 8.17 mm, vias 0 -> 1
- net Net-(JP3-A): track 8.15 -> 5.31 mm
- net SIM7080G_RTS: track 21.4 -> 18.9 mm, vias 1 -> 2
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- removed copper zone on In2.Cu, net GND
